File: watch.kicad_pcb (KiCad board)
At the start: 2 copper layers, 34.4 x 41.7 mm, 15 parts

Commit message: Correct pad numbers
Parts:
- REF**: footprint w_smd_leds:DUAL_LED -> DUAL_LED

Commit message: Are finished yet? I think we are...
Parts:
- added C1: C, w_smd_cap:c_0402, F.Cu at (-4.40, 0.25)
- added C2: C, w_smd_cap:c_0603, B.Cu at (-3.68, 12.3)
- added C3: C, w_smd_cap:c_0402, F.Cu at (4.19, 1.27)
- added G***: LOGO, w_logo:Logo_soldermask_OSHW_6x6mm, F.Cu at (0.00, 6.60)
- added PIN_SOCKET_2MM_3x2: Val**, w_pin_strip:pin_socket_2mm_3x2, B.Cu at (11.8, 2.54)
- added R1: R, w_smd_resistors:r_0603, B.Cu at (-3.56, -12.2)
- added R2: R, w_smd_resistors:r_0603, B.Cu at (13.0, -2.67)
- added R3: R, w_smd_resistors:r_0603, B.Cu at (13.0, -1.52)
- D1, D10, D11, D12, D2, D3, D4, D5, D6, D7, D8, D9: renamed from REF**; value LED-0603 -> LED_DUAL
- IC1: renamed from REF**; value QFN-32-1EP_5x5mm_Pitch0.5mm -> ATMEGA48A-M
- X1: renamed from c_1206; value C*** -> CRYSTAL
- moved X1 1.47 mm to (-5.59, 2.54), turned to 180 degrees
- turned D1 to 240 degrees
- turned D10 to 330 degrees
- turned D11 to 300 degrees
- turned D12 to 270 degrees
- turned D2 to 210 degrees
- turned D3 to 180 degrees
- turned D4 to 150 degrees
- turned D5 to 120 degrees
- turned D6 to 90 degrees
- turned D7 to 60 degrees
- turned D8 to 30 degrees
- turned D9 to 0 degrees
Connections:
- BT1 pad 1: (no net) -> GND
- BT1 pad 2: (no net) -> VCC
- D1 pad 1: (no net) -> /LED01
- D1 pad 2: (no net) -> /CATHODE_COLOR1
- D1 pad 3: (no net) -> /LED01
- D1 pad 4: (no net) -> /CATHODE_COLOR2
- D10 pad 1: (no net) -> /LED10
- D10 pad 2: (no net) -> /CATHODE_COLOR1
- D10 pad 3: (no net) -> /LED10
- D10 pad 4: (no net) -> /CATHODE_COLOR2
- D11 pad 1: (no net) -> /LED11
- D11 pad 2: (no net) -> /CATHODE_COLOR1
- D11 pad 3: (no net) -> /LED11
- D11 pad 4: (no net) -> /CATHODE_COLOR2
- D12 pad 1: (no net) -> /LED12
- D12 pad 2: (no net) -> /CATHODE_COLOR1
- D12 pad 3: (no net) -> /LED12
- D12 pad 4: (no net) -> /CATHODE_COLOR2
- D2 pad 1: (no net) -> /LED02
- D2 pad 2: (no net) -> /CATHODE_COLOR1
- D2 pad 3: (no net) -> /LED02
- D2 pad 4: (no net) -> /CATHODE_COLOR2
- D3 pad 1: (no net) -> /LED03
- D3 pad 2: (no net) -> /CATHODE_COLOR1
- D3 pad 3: (no net) -> /LED03
- D3 pad 4: (no net) -> /CATHODE_COLOR2
- D4 pad 1: (no net) -> /LED04
- D4 pad 2: (no net) -> /CATHODE_COLOR1
- D4 pad 3: (no net) -> /LED04
- D4 pad 4: (no net) -> /CATHODE_COLOR2
- D5 pad 1: (no net) -> /LED05
- D5 pad 2: (no net) -> /CATHODE_COLOR1
- D5 pad 3: (no net) -> /LED05
- D5 pad 4: (no net) -> /CATHODE_COLOR2
- D6 pad 1: (no net) -> /LED06
- D6 pad 2: (no net) -> /CATHODE_COLOR1
- D6 pad 3: (no net) -> /LED06
- D6 pad 4: (no net) -> /CATHODE_COLOR2
- D7 pad 1: (no net) -> /LED07
- D7 pad 2: (no net) -> /CATHODE_COLOR1
- D7 pad 3: (no net) -> /LED07
- D7 pad 4: (no net) -> /CATHODE_COLOR2
- D8 pad 1: (no net) -> /LED08
- D8 pad 2: (no net) -> /CATHODE_COLOR1
- D8 pad 3: (no net) -> /LED08
- D8 pad 4: (no net) -> /CATHODE_COLOR2
- D9 pad 1: (no net) -> /LED09
- D9 pad 2: (no net) -> /CATHODE_COLOR1
- D9 pad 3: (no net) -> /LED09
- D9 pad 4: (no net) -> /CATHODE_COLOR2
- IC1 pad 1: (no net) -> Net-(IC1-Pad1)
- IC1 pad 10: (no net) -> /LED07
- IC1 pad 11: (no net) -> /LED06
- IC1 pad 12: (no net) -> /LED05
- IC1 pad 13: (no net) -> /LED04
- IC1 pad 14: (no net) -> Net-(IC1-Pad14)
- IC1 pad 15: (no net) -> /MOSI
- IC1 pad 16: (no net) -> /MISO
- IC1 pad 17: (no net) -> /SCK
- IC1 pad 18: (no net) -> VCC
- IC1 pad 19: (no net) -> Net-(IC1-Pad19)
- IC1 pad 2: (no net) -> /LED09
- IC1 pad 20: (no net) -> Net-(C4-Pad1)
- IC1 pad 21: (no net) -> GND
- IC1 pad 22: (no net) -> Net-(IC1-Pad22)
- IC1 pad 23: (no net) -> /LED03
- IC1 pad 24: (no net) -> Net-(IC1-Pad24)
- IC1 pad 25: (no net) -> Net-(IC1-Pad25)
- IC1 pad 26: (no net) -> /LED02
- IC1 pad 27: (no net) -> /LED01
- IC1 pad 28: (no net) -> /LED12
- IC1 pad 29: (no net) -> /RESET
- IC1 pad 3: (no net) -> GND
- IC1 pad 30: (no net) -> /LED11
- IC1 pad 31: (no net) -> /LED10
- IC1 pad 32: (no net) -> Net-(IC1-Pad32)
- IC1 pad 33: (no net) -> GND
- IC1 pad 4: (no net) -> VCC
- IC1 pad 5: (no net) -> GND
- IC1 pad 6: (no net) -> VCC
- IC1 pad 7: (no net) -> Net-(IC1-Pad7)
- IC1 pad 8: (no net) -> Net-(IC1-Pad8)
- IC1 pad 9: (no net) -> /LED08
- X1 pad 1: (no net) -> Net-(IC1-Pad7)
- X1 pad 2: (no net) -> Net-(IC1-Pad8)
Routing:
- net /CATHODE_COLOR1: track 0.00 -> 149.6 mm, vias 0 -> 13
- net /CATHODE_COLOR2: track 0.00 -> 131.6 mm, vias 0 -> 12
- net VCC: track 0.00 -> 54.0 mm, vias 0 -> 2
- net /RESET: track 0.00 -> 34.1 mm, vias 0 -> 1
- net /MISO: track 0.00 -> 13.8 mm, vias 0 -> 1
- net /MOSI: track 0.00 -> 13.8 mm, vias 0 -> 1
- net /LED04: track 0.00 -> 12.7 mm
- net /SCK: track 0.00 -> 12.5 mm, vias 0 -> 1
- net /LED10: track 0.00 -> 11.5 mm
- net /LED02: track 0.00 -> 11.5 mm
- net /LED08: track 0.00 -> 11.4 mm
- net /LED05: track 0.00 -> 10.7 mm
- net Net-(IC1-Pad25): track 0.00 -> 10.6 mm, vias 0 -> 1
- net /LED11: track 0.00 -> 10.3 mm
- net /LED01: track 0.00 -> 10.3 mm
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- added copper zone on B.Cu, net GND
- added copper zone on F.Cu, net GND
Other:
- net class Default: clearance 0.254 -> 0.127; via_dia 0.889 -> 0.9; via_drill 0.635 -> 0.4
- rule trace_clearance: 0.254 -> 0.127
- rule via_min_drill: 0.508 -> 0.3
- rule via_min_size: 0.889 -> 0.6
- board text added: "g33kwatch v1.0 2015 mic@wemakethings.net (c) Albertas Mickėnas 2015"
